File: JO1_PCB.kicad_sch (KiCad schematic)
At the start: 21 parts, among them J1 CN8, J10 ESC_PWM, J11 CAN_WCMCU-1051_BLUEPILL, J13 LM2596_3.3V, J14 LM2596_5V, J2 CN7, J3 CN9, J4 CN10, J5 MPU-6050, J6 CAN_WCMCU-1051_NUCLEO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

Commit message: Routing
Parts:
- added J12: TFT, Connector_PinSocket_2.54mm:PinSocket_1x09_P2.54mm_Vertical, symbol Connector:Conn_01x09_Pin
- J13, J14: footprint (none) -> TerminalBlock_MetzConnect:TerminalBlock_MetzConnect_Type094_RT03502HBLU_1x02_P5.00mm_Horizontal
Connections:
- net 3.3V: now also U2.3V3 (3.3V), J12.2 (LED), J12.9 (VCC)
- net BLUEPILL_ENCODER_A: now also U2.PA0
- net BLUEPILL_ENCODER_B: now also U2.PA1
- net GND: now also J1.GND (13), J2.GND (8), J3.GND (23), J4.GND (5), U2.G (GND), J12.8 (GND)
- net BLUEPILL_TFT_RESET: now reaches U2.PA4
- net BLUEPILL_TFT_RESET: now also J12.6 (RESET)
- net BLUEPILL_TFT_CLK: now reaches U2.PA5
- net BLUEPILL_TFT_CLK: now also J12.3 (SCK)
- net BLUEPILL_TFT_DC: now reaches U2.PA6
- net BLUEPILL_TFT_DC: now also J12.5 (DC)
- net BLUEPILL_TFT_MOSI: now reaches U2.PA7
- net BLUEPILL_TFT_MOSI: now also J12.4 (MOSI)
- net BLUEPILL_TFT_CS: now reaches U2.PB0
- net BLUEPILL_TFT_CS: now also J12.7 (CS)
- no-connect marks 12 -> 121
Other:
- moved on the sheet: J13, J14, U2

Commit message: ya mero casi
Parts:
- added C1: 100nF, Capacitor_THT:C_Disc_D4.7mm_W2.5mm_P5.00mm, symbol Device:C_Small
- added R3: 1K, Resistor_THT:R_Axial_DIN0207_L6.3mm_D2.5mm_P10.16mm_Horizontal, symbol Device:R
- added SW1: SW_Nidec_CAS-120A1, Button_Switch_THT:SW_Slide-03_Wuerth-WS-SLTV_10x2.5x6.4_P2.54mm, symbol Switch:SW_Nidec_CAS-120A1
- R1, R2: footprint Resistor_THT:R_Axial_DIN0204_L3.6mm_D1.6mm_P5.08mm_Horizontal -> Resistor_THT:R_Axial_DIN0207_L6.3mm_D2.5mm_P10.16mm_Horizontal
Connections:
- net 3.3V: now also SW1.1 (C)
- net GND: now also C1.1, SW1.3 (A)
- net CAN_+: now reaches J11.5 (CANH), J6.5 (CANH), R1.2, R2.2
- net CAN_-: now reaches J11.6 (CANL), J6.6 (CANL), R1.1, R2.1
- net at J2.PB8 (2): now also C1.2, R3.2
- new net: R3.1, SW1.2 (B)
- no-connect marks 121 -> 120

Commit message: Version Nov 21
Connections:
- net GND: now also C1.2; no longer C1.1
- net at J2.PB8 (2), R3.2: now also C1.1; no longer C1.2
Other:
- moved on the sheet: C1, J1, J10, J11, J12, J13, J14, J2, J3, J4, J5, J6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

Commit message: Modified SPI
Connections:
- net NUCLEO_NRF_SPI5_MISO: no longer J3.PF8 (24)
- net NUCLEO_NRF_SPI5_MOSI: no longer J3.PF11 (11)
- net NUCLEO_NRF_SPI5_SCK: no longer J3.PF7 (26)
- net NUCLEO_NRF_SPI4_SCK: now reaches J3.PE2 (14)
- net NUCLEO_NRF_SPI4_MISO: now reaches J3.PE5 (18)
- net NUCLEO_NRF_SPI4_MOSI: now reaches J3.PE6 (20)
