File: JO1_PCB.kicad_pcb (KiCad board)
At the start: 2 copper layers, 59.5 x 78 mm, 21 parts, among them J1 CN8, J10 ESC_PWM, J11 CAN_WCMCU-1051_BLUEPILL, J12 TFT, J13 LM2596_3.3V, J14 LM2596_5V, J2 CN7, J3 CN9, J4 CN10, J5 MPU-6050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

Commit message: Final revision
Parts:
- added H1: MountingHole, MountingHole:MountingHole_2.1mm, F.Cu at (2.38, 2.38)
- added H2: MountingHole, MountingHole:MountingHole_2.1mm, F.Cu at (2.38, 8.12)
- added H3: MountingHole, MountingHole:MountingHole_2.1mm, F.Cu at (2.38, 13.9)
- added H4: MountingHole, MountingHole:MountingHole_2.1mm, F.Cu at (2.38, 19.6)
