File: JO1_PCB/JO1_PCB.kicad_pcb (KiCad board)
At the start: 2 copper layers, 66 x 80.7 mm, 23 parts, among them J1 CN8, J10 MCP2515_SPI, J11 MCP2515_CAN, J12 LM2596_3.3V, J13 LM2596_5V, J14 7.4V, J2 CN7, J3 CN9, J4 CN10, J5 DC_MOTOR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

Commit message: Routed PCB
Parts:
- added G***: LOGO, FOOTPRINTS:catlogo, F.Cu at (152.7, 107.6)
- moved M1 58.9 mm to (147.7, 125.7), turned to 90 degrees
- moved J7 40.0 mm to (140.3, 90.0), turned to 0 degrees
- moved BZ1 22.9 mm to (110.5, 93.0), turned to 90 degrees
- moved U1 6.99 mm to (133.0, 78.6), turned to -90 degrees
- moved R1 5.08 mm to (110.5, 104.9)
- moved J11 4.97 mm to (147.7, 120.9)
- moved J9 4.90 mm to (141.9, 131.0)
- moved J5 3.01 mm to (140.4, 70.1)
- moved J6 2.89 mm to (135.8, 72.6)
- moved A1 0.65 mm to (144.9, 61.7)
- moved J13 0.36 mm to (140.3, 61.9)
- moved J14 0.35 mm to (118.0, 61.9)
- moved J12 0.32 mm to (129.2, 61.9)
Connections:
- net CAN_+ renamed CAN_H
- net CAN_- renamed CAN_L
- J2 pad PC7: NUCLEO_NRF_CSN -> unconnected-(J2-11-PadPC7)
- J3 pad PE3: unconnected-(J3-22-PadPE3) -> NUCLEO_NRF_CSN
Routing:
- net NUCLEO_SERVO_TIM13_CH1: track 0.00 -> 82.8 mm
- net NUCLEO_NRF_CE: track 0.00 -> 65.2 mm
- net ARDUINO_NANO_SPI_INT: track 0.00 -> 64.0 mm
- net NUCLEO_NRF_SPI5_MISO: track 0.00 -> 43.6 mm
- net NUCLEO_NRF_CSN: track 0.00 -> 39.3 mm
- net NUCLEO_ESC_TIM14_CH1: track 0.00 -> 37.1 mm
- net NUCLEO_NRF_SPI5_SCK: track 0.00 -> 35.9 mm
- net NUCLEO_FDCAN_RX: track 0.00 -> 35.6 mm
- net NUCLEO_NRF_SPI5_MOSI: track 0.00 -> 34.9 mm
- net ARDUINO_NANO_SPI_MOSI: track 0.00 -> 34.6 mm
- net NUCLEO_FDCAN_TX: track 0.00 -> 30.7 mm
- net ARDUINO_NANO_SPI_CS: track 0.00 -> 30.5 mm
- net ARDUINO_NANO_SPI_MISO: track 0.00 -> 27.5 mm
- net ARDUINO_NANO_SPI_SCK: track 0.00 -> 27.1 mm
- net 7.4V: track 0.00 -> 25.8 mm
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- added copper zone on F.Cu, net 5V
Other:
- board text added: "CEJ2 Robotics"
- board text added: "NUCLEO-H745ZI-Q Shield"

Commit message: Added visual indications
Parts:
- added G***: LOGO, FOOTPRINTS:star, F.Cu at (111.3, 108.1)
- added G***: LOGO, FOOTPRINTS:joebiden, F.Cu at (152.5, 76.8)
- added G***: LOGO, FOOTPRINTS:star, F.Cu at (160.4, 108.0)
- added G***: LOGO, FOOTPRINTS:star, F.Cu at (144.7, 131.2)
- added G***: LOGO, FOOTPRINTS:star, F.Cu at (142.8, 70.0)
- added G***: LOGO, FOOTPRINTS:johndeerelogo, F.Cu at (111.6, 73.5)
- added G***: LOGO, FOOTPRINTS:star, F.Cu at (138.1, 69.9)
- added G***: LOGO, FOOTPRINTS:star, F.Cu at (147.7, 124.2)
- added G***: LOGO, FOOTPRINTS:star, F.Cu at (142.7, 95.1)
Other:
- board text added: "+"
- board text added: "-"
- board text added: "3.3V"
- board text added: "5V"
- board text added: "7.4V"
- board text added: "ARDUINO NANO"
- board text added: "CAN_H"
- board text added: "CAN_L"
- board text added: "DC_MOTOR"
- board text added: "ESC_MOTOR"
- board text added: "ESC_PWM"
- board text added: "MCP2515_CAN"
- board text added: "MCP2515_SPI"
- board text added: "MPU6050"
- board text added: "NRF24L01"
- board text added: "SERVO"
- board text added: "TJA1051"
- board text added: "github.com/CEJ2-Robotics/JO1_Electronics v1.0.0"

Commit message: Added text
Parts:
- added G***: LOGO, FOOTPRINTS:teclogo, F.Cu at (111.6, 76.2)
- moved G*** 2.67 mm to (111.7, 70.8)
